File: USBChargerDIY/kicad/typeC/typeC.kicad_sch (KiCad schematic)
At the start: 16 parts, among them J1 USB_C_Receptacle_USB2.0_14P, U1 TLP785, U2 HA17339A, U3 HA17339A, U4 TLP785

Commit message: update
Connections:
- net at U4.2: now also U2.1; no longer U3.1
- net at U1.2: now also U3.1; no longer U2.1
Changed lines of the file:
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@@
     (stroke (width 0) (type default) (color 0 0 0 1))
+  )
+  (wire (pts (xy 95.25 87.63) (xy 119.38 87.63))
+    (stroke (width 0) (type default))
   )
   (wire (pts (xy 116.84 58.42) (xy 130.81 58.42))
@@
     (stroke (width 0) (type default))
   )
+  (wire (pts (xy 119.38 87.63) (xy 119.38 95.25))
+    (stroke (width 0) (type default))
+  )
   (wire (pts (xy 82.55 58.42) (xy 116.84 58.42))
     (stroke (width 0) (type default) (color 194 0 0 1))
@@
     (stroke (width 0) (type default))
   )
+  (wire (pts (xy 92.71 93.98) (xy 92.71 69.85))
+    (stroke (width 0) (type default))
+  )
   (wire (pts (xy 82.55 92.71) (xy 82.55 97.79))
     (stroke (width 0) (type default))
@@
     (stroke (width 0) (type default) (color 194 0 0 1))
   )
-  (wire (pts (xy 95.25 87.63) (xy 95.25 93.98))
-    (stroke (width 0) (type default))
-  )
   (wire (pts (xy 71.12 97.79) (xy 71.12 100.33))
     (stroke (width 0) (type default))
@@
     (stroke (width 0) (type default))
   )
-  (wire (pts (xy 119.38 95.25) (xy 119.38 87.63))
-    (stroke (width 0) (type default))
-  )
   (wire (pts (xy 161.29 72.39) (xy 161.29 78.74))
     (stroke (width 0) (type default))
   )
+  (wire (pts (xy 140.97 69.85) (xy 140.97 78.74))
+    (stroke (width 0) (type default))
+  )
   (wire (pts (xy 87.63 107.95) (xy 82.55 107.95))
     (stroke (width 0) (type default) (color 0 0 0 1))
@@
     (stroke (width 0) (type default))
   )
+  (wire (pts (xy 92.71 69.85) (xy 140.97 69.85))
+    (stroke (width 0) (type default))
+  )
   (wire (pts (xy 87.63 97.79) (xy 82.55 97.79))
     (stroke (width 0) (type default))
@@
     (stroke (width 0) (type default))
   )
-  (wire (pts (xy 119.38 87.63) (xy 95.25 87.63))
+  (wire (pts (xy 95.25 80.01) (xy 95.25 87.63))
     (stroke (width 0) (type default))
   )
@@
     (stroke (width 0) (type default))
   )
-  (wire (pts (xy 95.25 69.85) (xy 140.97 69.85))
-    (stroke (width 0) (type default))
-  )
   (wire (pts (xy 110.49 82.55) (xy 110.49 86.36))
     (stroke (width 0) (type default))
@@
     (stroke (width 0) (type default))
   )
-  (wire (pts (xy 140.97 69.85) (xy 140.97 78.74))
-    (stroke (width 0) (type default))
-  )
   (wire (pts (xy 130.81 58.42) (xy 138.43 58.42))
     (stroke (width 0) (type default) (color 194 0 0 1))
   )
+  (wire (pts (xy 95.25 93.98) (xy 92.71 93.98))
+    (stroke (width 0) (type default))
+  )
   (wire (pts (xy 138.43 68.58) (xy 138.43 91.44))
     (stroke (width 0) (type default))
@@
     (stroke (width 0) (type default))
   )
-  (wire (pts (xy 95.25 80.01) (xy 95.25 69.85))
-    (stroke (width 0) (type default))
-  )
