File: KitchenTimer/pic_version/kicad/TimerPIC12F1840_1/TimerPIC12F1840_1.kicad_sch (KiCad schematic)
At the start: 18 parts, among them SW1 SW_DIP_x04, SW2 SW_SPST, SW3 SW_SPST, SW4 SW_SPST, SW5 SW_SPST

Commit message: update
Parts:
- removed ArduinoUnoR1: ~, symbol Ore:ArduinoUnoR3
- removed R1, R2, R3, R4, R5: R, symbol Device:R
- removed SW1: SW_DIP_x04, symbol Switch:SW_DIP_x04
Other:
- moved on the sheet: LS1, MU1, R1, R2, R3, R4, R5

Commit message: update
Parts:
- added SW1: SW_Push, symbol Switch:SW_Push
- renumbered R4 to R2, R2 to R4
Connections:
- net at R2.1, SW5.2 (B): now also MU1.6 (RA1); no longer MU1.5 (RA2)
- net at LS1.2, MU1.8 (VSS), R2.2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: now also SW1.2
- net at R3.1, SW4.2 (B): now also MU1.5 (RA2); no longer MU1.4 (RA3)
- new net: MU1.4 (RA3), SW1.1
Other:
- moved on the sheet: R2, R3, R4, R5
