File: USBHub/MA8601/kicad/MA8601_v1.0/MA8601_v1.0.kicad_sch (KiCad schematic)
At the start: 11 parts, among them J1 USB_B, Q1 PMOS, Q2 NMOS, Q3 NMOS, SW1 SW_DPDT_x2, SW2 SW_DIP_x01, Y1 Crystal

Commit message: update
Parts:
- removed Q1: PMOS, symbol Simulation_SPICE:PMOS
- removed Q2, Q3: NMOS, symbol Simulation_SPICE:NMOS
- removed SW2: SW_DIP_x01, symbol Switch:SW_DIP_x01
- added C3: 1uF, symbol Device:C
- added C4: 470uF, symbol Device:C_Polarized
- added C5, C6, C7: 10uF, symbol Device:C
- added J2, J3, J4, J5: USB_A femele connector, symbol Connector:USB_A
- added R1: 300 ohm, symbol Device:R
- C1, C2: value C -> 15pF
- J1: value USB_B -> USB_B Female connector
- R2: value R -> 10k ohm
- SW1: value SW_DPDT_x2 -> M-2022NB
- U1: value ~ -> MA8601
- Y1: value Crystal -> crystal 12MHz
Connections:
- net GND: now also C3.2, C4.2, C5.2, C6.2, C7.2, J2.4 (GND), J2.5 (Shield), J3.4 (GND), J3.5 (Shield), J4.4 (GND), J4.5 (Shield), J5.4 (GND), J5.5 (Shield), R1.1; no longer R2.2
- net PSELF: no longer R2.1
- net VCC1V2: now also C7.1
- net VCC3V3: now also R2.1, U1.26 (OVCJ), C6.1
- net VCC5V: now also C4.1, C5.1, J2.1 (VBUS), J3.1 (VBUS), J4.1 (VBUS), J5.1 (VBUS)
- net DM1: now reaches U1.10 (DM1)
- net DM1: now also J2.2 (D-)
- net DP1: now reaches U1.11 (DP1)
- net DP1: now also J2.3 (D+)
- net at U1.14 (REXT): now also R1.2
- net SRST: now reaches U1.17 (SRST)
- net SRST: now also R2.2, C3.1
- net DM4: now reaches U1.4 (DM4)
- net DM4: now also J5.2 (D-)
- net DP4: now reaches U1.5 (DP4)
- net DP4: now also J5.3 (D+)
- net DM3: now reaches U1.6 (DM3)
- net DM3: now also J4.2 (D-)
- net DP3: now reaches U1.7 (DP3)
- net DP3: now also J4.3 (D+)
- net DM2: now reaches U1.8 (DM2)
- net DM2: now also J3.2 (D-)
- net DP2: now reaches U1.9 (DP2)
- net DP2: now also J3.3 (D+)
- no-connect marks 0 -> 5
Other:
- note added: "Self powr selector."
- note removed: "It does not work!!!"
- note removed: "Self power selector plan A."
- note removed: "Self powr selector plan B."
- moved on the sheet: C1, C2, J1, SW1A, U1, Y1
