File: CondenserMeasure/kicad/AutoRegisterSelectorEdition1.0/AutoRegisterSelectorEdition1.0.kicad_sch (KiCad schematic)
At the start: 6 parts, among them U1 ATmega328P

Commit message: update
Parts:
- R2: value 10k -> 22k
Changed lines of the file:
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@@
       (effects (font (size 1.27 1.27)) (justify left))
     )
-    (property "Value" "10k" (at 52.07 77.47 0)
+    (property "Value" "22k" (at 52.07 77.47 0)
       (effects (font (size 1.27 1.27)) (justify left))
     )
