File: USBHub/GL850G/kicad/GL850G_2.0/GL850G_2.0.kicad_sch (KiCad schematic)
At the start: 14 parts, among them J1 USB_B Female connector, J2 USB_A femele connector, J3 USB_A femele connector, J4 USB_A femele connector, J5 USB_A femele connector, SW1 SW_SPDT, U1 GL850G, Y1 12MHz

Commit message: update
Connections:
- net GND: no longer U1.17 (PSELF)
- net V33: now also U1.17 (PSELF)
Changed lines of the file:
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@@
-		)
-	)
-	(wire
-		(pts
-			(xy 83.82 85.09) (xy 92.71 85.09)
-		)
-		(stroke
-			(width 0)
-			(type default)
 		)
 	)
@@
 		(property "Intersheetrefs" "${INTERSHEET_REFS}"
 			(at 127.5661 113.03 0)
+			(effects
+				(font
+					(size 1.27 1.27)
+				)
+				(justify left)
+				(hide yes)
+			)
+		)
+	)
+	(global_label "V33"
+		(shape input)
+		(at 83.82 85.09 0)
+		(fields_autoplaced yes)
+		(effects
+			(font
+				(size 1.27 1.27)
+			)
+			(justify left)
+		)
+		(property "Intersheetrefs" "${INTERSHEET_REFS}"
+			(at 90.3128 85.09 0)
 			(effects
 				(font
@@
 					(unit 1)
 				)
-			)
-		)
-	)
-	(symbol
-		(lib_name "GND_1")
-		(lib_id "power:GND")
-		(at 92.71 85.09 0)
-		(unit 1)
-		(exclude_from_sim no)
-		(in_bom yes)
-		(on_board yes)
-		(dnp no)
-		(fields_autoplaced yes)
-		(property "Reference" "#PWR07"
-			(at 92.71 91.44 0)
-			(effects
-				(font
-					(size 1.27 1.27)
-				)
-				(hide yes)
-			)
-		)
-		(property "Value" "GND"
-			(at 92.71 90.17 0)
-			(effects
-				(font
-					(size 1.27 1.27)
-				)
-			)
-		)
-		(property "Footprint" ""
-			(at 92.71 85.09 0)
-			(effects
-				(font
-					(size 1.27 1.27)
-				)
-				(hide yes)
-			)
-		)
-		(property "Datasheet" ""
-			(at 92.71 85.09 0)
-			(effects
-				(font
-					(size 1.27 1.27)
-				)
-				(hide yes)
-			)
-		)
-		(property "Description" "Power symbol creates a global label with name \"GND\" , ground"
-			(at 92.71 85.09 0)
-			(effects
-				(font
-					(size 1.27 1.27)
-				)
-				(hide yes)
-			)
-		)
-		(pin "1"
-		)
-		(instances
-			(project "GL850G_2.0"
-				(path "/ddc50684-2832-457a-af57-346958dc495f"
-					(reference "#PWR07")
-					(unit 1)
-				)

Commit message: update
Parts:
- C3: value 0.1u -> 1u
Changed lines of the file:
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@@
+		)
+	)
+	(text_box "実際にはスイッチではなくて単に\nターミナルに使いたい方を差すだけ。"
+		(exclude_from_sim no)
+		(at 43.18 22.86 0)
+		(size 30.48 5.08)
+		(stroke
+			(width 0)
+			(type default)
+		)
+		(fill
+			(type none)
+		)
+		(effects
+			(font
+				(face "源ノ角ゴシック Code JP M")
+				(size 1.27 1.27)
+			)
+			(justify left top)
 		)
 	)
@@
 			)
 		)
-		(property "Value" "0.1u"
+		(property "Value" "1u"
 			(at 105.41 58.166 0)
 			(effects
