File: USBSwitcher/TC7USB40FT/kicad/TC7USB40FT_1.0/TC7USB40FT_1.0.kicad_sch (KiCad schematic)
At the start: 11 parts, among them J1 USB_B, J2 USB_A, J3 USB_B, SW1 2回路トグルスイッチ, U1 NJM2845DL1-33, U2 TC7USB40FT

Commit message: update
Parts:
- renumbered J3 to J2, J2 to J3
Changed lines of the file:
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@@
 		)
 	)
-	(text_box "C1: 100uF 前後で OK\nC2: 0.33uF 以上で多分 OK"
+	(text_box "C1: Roughly 100uF\nC2: C2 >= 0.33uF, Ceramic\nC3: C3 >= 2.2uF, Ceramic"
 		(exclude_from_sim no)
 		(at 88.9 96.52 0)
@@
 		(dnp no)
 		(fields_autoplaced yes)
-		(property "Reference" "J3"
+		(property "Reference" "J2"
 			(at 43.18 16.51 0)
 			(effects
@@
 			(project ""
 				(path "/e15c2708-3073-48fd-862b-d302223bf0d2"
-					(reference "J3")
+					(reference "J2")
 					(unit 1)
 				)
@@
 		(dnp no)
 		(fields_autoplaced yes)
-		(property "Reference" "J2"
+		(property "Reference" "J3"
 			(at 24.13 83.82 0)
 			(effects
@@
 			(project ""
 				(path "/e15c2708-3073-48fd-862b-d302223bf0d2"
-					(reference "J2")
+					(reference "J3")
 					(unit 1)
 				)
