File: PS_2-to-USB_KB/kicad/ps2-USB_KB_1.1/ps2-USB_KB_1.1.kicad_sch (KiCad schematic)
At the start: 4 parts, among them J1 USB_B, U1 PIC16F1455

Commit message: update
Parts:
- added SW1: SW_DIP_x01, symbol Switch:SW_DIP_x01
Connections:
- net 5V: now also SW1.2; no longer C1.1, J1.1 (VBUS)
- new net: C1.1, J1.1 (VBUS), SW1.1
Changed lines of the file:
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@@
 	(paper "A5" portrait)
 	(junction
-		(at 69.85 36.83)
+		(at 97.79 35.56)
 		(diameter 0)
 		(color 0 0 0 0)
@@
 	(wire
 		(pts
+			(xy 43.18 25.4) (xy 49.53 25.4)
+		)
+		(stroke
+			(width 0)
+			(type default)
+		)
+	)
+	(wire
+		(pts
+			(xy 64.77 25.4) (xy 68.58 25.4)
+		)
+		(stroke
+			(width 0)
+			(type default)
+		)
+	)
+	(wire
+		(pts
 			(xy 22.86 40.64) (xy 25.4 40.64)
 		)
@@
 	(wire
 		(pts
-			(xy 63.5 31.75) (xy 69.85 31.75)
-		)
-		(stroke
-			(width 0)
-			(type default)
-		)
-	)
-	(wire
-		(pts
-			(xy 45.72 25.4) (xy 43.18 25.4)
+			(xy 91.44 30.48) (xy 97.79 30.48)
 		)
 		(stroke
@@
 	(wire
 		(pts
-			(xy 69.85 31.75) (xy 69.85 36.83)
+			(xy 97.79 30.48) (xy 97.79 35.56)
 		)
 		(stroke
@@
 	(wire
 		(pts
-			(xy 63.5 36.83) (xy 69.85 36.83)
+			(xy 91.44 35.56) (xy 97.79 35.56)
 		)
 		(stroke
@@
 	(text "KB: JKB-89S"
 		(exclude_from_sim no)
-		(at 64.516 22.352 0)
+		(at 92.456 21.082 0)
 		(effects
 			(font
@@
 	(global_label "KBD_CLK"
 		(shape input)
-		(at 63.5 26.67 0)
+		(at 91.44 25.4 0)
 		(fields_autoplaced yes)
 		(effects
@@
 		)
 		(property "Intersheetrefs" "${INTERSHEET_REFS}"
-			(at 74.8309 26.67 0)
+			(at 102.7709 25.4 0)
 			(effects
 				(font
@@
 	(global_label "5V"
 		(shape input)
-		(at 45.72 25.4 0)
+		(at 68.58 25.4 0)
 		(fields_autoplaced yes)
 		(effects
@@
 		)
 		(property "Intersheetrefs" "${INTERSHEET_REFS}"
-			(at 51.0033 25.4 0)
+			(at 73.8633 25.4 0)
 			(effects
 				(font
@@
 	(global_label "KBD_DATA"
 		(shape input)
-		(at 63.5 29.21 0)
+		(at 91.44 27.94 0)
 		(fields_autoplaced yes)
 		(effects
@@
 		)
 		(property "Intersheetrefs" "${INTERSHEET_REFS}"
-			(at 75.6776 29.21 0)
+			(at 103.6176 27.94 0)
 			(effects
 				(font
@@
 	(global_label "5V"
 		(shape input)
-		(at 63.5 34.29 0)
+		(at 91.44 33.02 0)
 		(fields_autoplaced yes)
 		(effects
@@
 		)
 		(property "Intersheetrefs" "${INTERSHEET_REFS}"
-			(at 68.7833 34.29 0)
+			(at 96.7233 33.02 0)
 			(effects
 				(font
@@
 		(length 2.54)
 		(shape round)
-		(at 63.5 29.21 90)
+		(at 91.44 27.94 90)
 		(effects
 			(font
@@
 		)
 		(property "Netclass" "Data"
-			(at 55.118 29.21 0)
+			(at 83.058 27.94 0)
 			(effects
 				(font
@@
 		(length 2.54)
 		(shape round)
-		(at 63.5 26.67 90)
+		(at 91.44 25.4 90)
 		(effects
 			(font
@@
 		)
 		(property "Netclass" "Clock"
-			(at 54.356 26.416 0)
+			(at 82.296 25.146 0)
 			(effects
 				(font
@@
 		(length 2.54)
 		(shape round)
-		(at 63.5 36.83 90)
+		(at 91.44 35.56 90)
 		(effects
 			(font
@@
 		)
 		(property "Netclass" "Shield"
-			(at 53.34 36.576 0)
+			(at 81.28 35.306 0)
 			(effects
 				(font
@@
 		(length 2.54)
 		(shape round)
-		(at 63.5 34.29 90)
+		(at 91.44 33.02 90)
 		(effects
 			(font
@@
 		)
 		(property "Netclass" "5V"
-			(at 57.15 34.29 0)
+			(at 85.09 33.02 0)
 			(effects
 				(font
@@
 		(length 2.54)
 		(shape round)
-		(at 63.5 31.75 90)
+		(at 91.44 30.48 90)
 		(effects
 			(font
@@
 		)
 		(property "Netclass" "GND"
-			(at 55.88 32.004 0)
+			(at 83.82 30.734 0)
 			(effects
 				(font
@@
 	)
 	(symbol
-		(lib_id "power:GND")
-		(at 69.85 36.83 0)
+		(lib_id "Switch:SW_DIP_x01")
+		(at 57.15 25.4 0)
 		(unit 1)
 		(exclude_from_sim no)
@@
 		(on_board yes)
 		(dnp no)
+		(property "Reference" "SW1"
+			(at 57.15 21.082 0)
+			(effects
+				(font
+					(size 1.27 1.27)
+				)
+			)
+		)
+		(property "Value" "SW_DIP_x01"
+			(at 57.15 20.32 0)
+			(effects
+				(font
+					(size 1.27 1.27)
+				)
+				(hide yes)
+			)
+		)
+		(property "Footprint" ""
+			(at 57.15 25.4 0)
+			(effects
+				(font
+					(size 1.27 1.27)
+				)
+				(hide yes)
+			)
+		)
+		(property "Datasheet" "~"
+			(at 57.15 25.4 0)
+			(effects
+				(font
+					(size 1.27 1.27)
+				)
+				(hide yes)
+			)
+		)
+		(property "Description" "1x DIP Switch, Single Pole Single Throw (SPST) switch, small symbol"
+			(at 57.15 25.4 0)
+			(effects
+				(font
+					(size 1.27 1.27)
+				)
+				(hide yes)
+			)
+		)
+		(pin "1"
+		)
+		(pin "2"
+		)
+		(instances
+			(project ""
+				(path "/736b408f-dea8-4e8d-8d76-24c6bbb1dde8"
+					(reference "SW1")
+					(unit 1)
+				)
+			)
+		)
+	)
+	(symbol
+		(lib_id "power:GND")
+		(at 97.79 35.56 0)
+		(unit 1)
+		(exclude_from_sim no)
+		(in_bom yes)
+		(on_board yes)
+		(dnp no)
 		(fields_autoplaced yes)
 		(property "Reference" "#PWR02"
-			(at 69.85 43.18 0)
+			(at 97.79 41.91 0)
 			(effects
 				(font
@@
 		)
 		(property "Value" "GND"
-			(at 69.85 41.91 0)
+			(at 97.79 40.64 0)
 			(effects
 				(font
@@
 		)
 		(property "Footprint" ""
-			(at 69.85 36.83 0)
+			(at 97.79 35.56 0)
 			(effects
 				(font
@@
 		)
 		(property "Datasheet" ""
-			(at 69.85 36.83 0)
+			(at 97.79 35.56 0)
 			(effects
 				(font
@@
 		)
 		(property "Description" "Power symbol creates a global label with name \"GND\" , ground"
-			(at 69.85 36.83 0)
-			(effects
-				(font
+			(at 97.79 35.56 0)
+			(effects
+				(font
