File: OreDuino_wo_Tsukuritai/kicad/ASOBoardR4_v1.1.1/ASOBoardR4_v1.1.1.kicad_sch (KiCad schematic)
At the start: 31 parts, among them J1 USB_B, J2 Conn_01x11_Socket, J3 Conn_01x14_Socket, J4 Conn_01x09_Socket, SW1 SW_Push

Commit message: update
Parts:
- removed C4, C7: 4.7u, symbol Device:C
- removed C5: 0.1u, symbol Device:C
- removed L2: 1.3u, symbol Device:L
- removed R4: 10k, symbol Device:R
Connections:
- net 5V: now also C8.1, U1.56 (AVCC)

Commit message: update
Parts:
- removed R7, R8, R9: 10k, symbol Device:R
Connections:
- net 3V3: now also U1.16 (USB_V); no longer U1.4 (VBAT)
- no-connect marks 0 -> 1

Commit message: update
Parts:
- removed R10: 100k, symbol Device:R
- removed R26: 13.7k, symbol Device:R
Connections:
- net GND: no longer J4.7 (Pin_7)
- net 49: now reaches U1.49
- net 49: now also J4.7 (Pin_7)
