File: CondenserMeasure/kicad/CapMeter3.0/CapMeter3.0.kicad_sch (KiCad schematic)
At the start: 8 parts, among them U1 ATmega328P, U2 LCD

Commit message: update
Parts:
- R1: value 75 -> 1k
- R2: value 22k -> 100k
- R4: value 200 -> 300
Changed lines of the file:
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@@
 			)
 		)
-		(property "Value" "75"
+		(property "Value" "1k"
 			(at 36.83 96.52 0)
 			(effects
@@
 			)
 		)
-		(property "Value" "200"
+		(property "Value" "300"
 			(at 36.83 77.47 0)
 			(effects
@@
 			)
 		)
-		(property "Value" "22k"
+		(property "Value" "100k"
 			(at 36.83 90.17 0)
 			(effects
