File: LuxMeter/v1.0/LuxMeter1.0/LuxMeter1.0.kicad_sch (KiCad schematic)
At the start: 6 parts, among them J1 Conn_01x04, J2 Conn_01x01, Q1 NJL7502L, SW1 SW_Push, U1 R7F101G6E2DSP Board

Commit message: update
Connections:
- net GND: now also R1.2
- net at U1.14 (P12): no longer R1.2
Other:
- moved on the sheet: Q1, R1
Changed lines of the file:
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@@
 	)
 	(junction
-		(at 97.79 40.64)
+		(at 97.79 48.26)
 		(diameter 0)
 		(color 0 0 0 0)
@@
 	(wire
 		(pts
-			(xy 88.9 40.64) (xy 97.79 40.64)
+			(xy 81.28 48.26) (xy 97.79 48.26)
 		)
 		(stroke
@@
 	(wire
 		(pts
-			(xy 81.28 50.8) (xy 97.79 50.8)
+			(xy 97.79 48.26) (xy 97.79 50.8)
 		)
 		(stroke
@@
 	(wire
 		(pts
-			(xy 81.28 48.26) (xy 88.9 48.26)
+			(xy 49.53 45.72) (xy 58.42 45.72)
 		)
 		(stroke
@@
 	(wire
 		(pts
-			(xy 97.79 40.64) (xy 97.79 43.18)
+			(xy 49.53 55.88) (xy 58.42 55.88)
 		)
 		(stroke
@@
 		)
 	)
-	(wire
-		(pts
-			(xy 49.53 45.72) (xy 58.42 45.72)
-		)
-		(stroke
-			(width 0)
-			(type default)
-		)
-	)
-	(wire
-		(pts
-			(xy 88.9 40.64) (xy 88.9 48.26)
-		)
-		(stroke
-			(width 0)
-			(type default)
-		)
-	)
-	(wire
-		(pts
-			(xy 49.53 55.88) (xy 58.42 55.88)
-		)
-		(stroke
-			(width 0)
-			(type default)
-		)
-	)
 	(global_label "SDA"
 		(shape input)
@@
 	(global_label "5V"
 		(shape input)
-		(at 97.79 30.48 90)
+		(at 97.79 38.1 90)
 		(fields_autoplaced yes)
 		(effects
@@
 		)
 		(property "Intersheetrefs" "${INTERSHEET_REFS}"
-			(at 97.79 25.3474 90)
+			(at 97.79 32.9674 90)
 			(effects
 				(font
@@
 				(justify left)
 				(hide yes)
+			)
+		)
+	)
+	(symbol
+		(lib_id "power:GND")
+		(at 97.79 58.42 0)
+		(unit 1)
+		(exclude_from_sim no)
+		(in_bom yes)
+		(on_board yes)
+		(dnp no)
+		(fields_autoplaced yes)
+		(property "Reference" "#PWR04"
+			(at 97.79 64.77 0)
+			(effects
+				(font
+					(size 1.27 1.27)
+				)
+				(hide yes)
+			)
+		)
+		(property "Value" "GND"
+			(at 97.79 63.5 0)
+			(effects
+				(font
+					(size 1.27 1.27)
+				)
+			)
+		)
+		(property "Footprint" ""
+			(at 97.79 58.42 0)
+			(effects
+				(font
+					(size 1.27 1.27)
+				)
+				(hide yes)
+			)
+		)
+		(property "Datasheet" ""
+			(at 97.79 58.42 0)
+			(effects
+				(font
+					(size 1.27 1.27)
+				)
+				(hide yes)
+			)
+		)
+		(property "Description" "Power symbol creates a global label with name \"GND\" , ground"
+			(at 97.79 58.42 0)
+			(effects
+				(font
+					(size 1.27 1.27)
+				)
+				(hide yes)
+			)
+		)
+		(pin "1"
+		)
+		(instances
+			(project "LuxMeter1.0"
+				(path "/29b11b00-85a1-4edc-9f3b-c77288705c4a"
+					(reference "#PWR04")
+					(unit 1)
+				)
 			)
 		)
@@
 	(symbol
 		(lib_id "Device:R")
-		(at 97.79 46.99 0)
+		(at 97.79 54.61 0)
 		(unit 1)
 		(exclude_from_sim no)
@@
 		(dnp no)
 		(property "Reference" "R1"
-			(at 99.314 45.212 0)
+			(at 99.314 52.832 0)
 			(effects
 				(font
@@
 		)
 		(property "Value" "10k"
-			(at 98.044 49.276 90)
+			(at 98.044 56.896 90)
 			(effects
 				(font
@@
 		)
 		(property "Footprint" ""
-			(at 96.012 46.99 90)
+			(at 96.012 54.61 90)
 			(effects
 				(font
@@
 		)
 		(property "Datasheet" "~"
-			(at 97.79 46.99 0)
+			(at 97.79 54.61 0)
 			(effects
 				(font
@@
 		)
 		(property "Description" "Resistor"
-			(at 97.79 46.99 0)
+			(at 97.79 54.61 0)
 			(effects
 				(font
@@
 	(symbol
 		(lib_id "Device:Q_Photo_NPN")
-		(at 95.25 35.56 0)
+		(at 95.25 43.18 0)
 		(unit 1)
 		(exclude_from_sim no)
@@
 		(fields_autoplaced yes)
 		(property "Reference" "Q1"
-			(at 100.33 32.9056 0)
+			(at 100.33 40.5256 0)
 			(effects
 				(font
@@
 		)
 		(property "Value" "NJL7502L"
-			(at 100.33 36.7156 0)
+			(at 100.33 44.3356 0)
 			(effects
 				(font
@@
 		)
 		(property "Footprint" ""
-			(at 100.33 33.02 0)
+			(at 100.33 40.64 0)
 			(effects
 				(font
@@
 		)
 		(property "Datasheet" "~"
-			(at 95.25 35.56 0)
+			(at 95.25 43.18 0)
 			(effects
 				(font
@@
 		)
 		(property "Description" "NPN phototransistor, collector/emitter"
-			(at 95.25 35.56 0)
-			(effects
-				(font
+			(at 95.25 43.18 0)
+			(effects
+				(font
